Commit message: pitched the kinect down to table

File: src/baxter_description/urdf/baxter.urdf.xacro (robot description, xacro)
@@ -27,5 +27,5 @@
     <xacro:include filename="$(find baxter_description)/urdf/sensors/kinect_camera.urdf.xacro" />
     <xacro:kinect_camera_v0 name="kinect_mount" parent="head">
-        <origin xyz="0.5 0.0 0.5" rpy="0 0 0" />
+        <origin xyz="0.5 0.0 0.5" rpy="0 45 0" />
     </xacro:kinect_camera_v0>
 </robot>

Commit message: moved kinect sensor to be centered over table

File: src/baxter_description/urdf/baxter.urdf.xacro (robot description, xacro)
@@ -27,5 +27,5 @@
     <xacro:include filename="$(find baxter_description)/urdf/sensors/kinect_camera.urdf.xacro" />
     <xacro:kinect_camera_v0 name="kinect_mount" parent="head">
-        <origin xyz="0.5 0.0 0.5" rpy="0 45 0" />
+        <origin xyz="0.93 0.0 0.34" rpy="0 1.57 0" />
     </xacro:kinect_camera_v0>
 </robot>

Commit message: move objs so baxter can reach them

File: src/baxter_description/urdf/baxter.urdf.xacro (robot description, xacro)
@@ -27,5 +27,5 @@
     <xacro:include filename="$(find baxter_description)/urdf/sensors/kinect_camera.urdf.xacro" />
     <xacro:kinect_camera_v0 name="kinect_mount" parent="head">
-        <origin xyz="0.93 0.0 0.34" rpy="0 1.57 0" />
+        <origin xyz="0.78 0.0 0.34" rpy="0 1.57 0" />
     </xacro:kinect_camera_v0>
 </robot>
